Commit message: fix bugs so that irg-raw3-6 is working with the real robot by comparing irg-backup-brad with irg-raw3-6. Now it works for web interface + teleop base

File: cob_description/urdf/drive_wheel/drive_wheel.urdf.xacro (robot description, xacro)
@@ -6,5 +6,7 @@
   <xacro:property name="caster_mass" value="5.9" />
   <xacro:property name="wheel_mass" value="0.44036" />
-  <xacro:macro name="cob_wheel" params="parent suffix reflect drive_vel:=^">
+  <!-- alpha tested effort and velocity limits -->
+  <!-- <xacro:macro name="cob_wheel" params="parent suffix reflect drive_vel:=^"> -->
+  <xacro:macro name="cob_wheel" params="parent suffix reflect drive_vel:=100">
     <joint name="${parent}_${suffix}_wheel_joint" type="continuous">
       <origin xyz="0 ${reflect*caster_wheel_offset_y} 0" rpy="0 0 0" />
@@ -39,5 +41,7 @@
   </xacro:macro>
   <!-- Macro for Caster hub only -->
-  <xacro:macro name="cob_caster_hub" params="*origin parent suffix steer_vel:=^" >
+  <!-- alpha tested velocity and effort limits -->
+  <!-- <xacro:macro name="cob_caster_hub" params="*origin parent suffix steer_vel:=^" > -->
+  <xacro:macro name="cob_caster_hub" params="*origin parent suffix steer_vel:=10" >
     <joint name="${suffix}_rotation_joint" type="continuous">
       <xacro:insert_block name="origin" />
@@ -71,5 +75,6 @@
     <xacro:cob_caster_transmission suffix="${suffix}" />
   </xacro:macro>
-  <xacro:macro name="drive_wheel" params="*origin parent suffix drive_vel:=^|100 steer_vel:=^|100">
+  <!-- <xacro:macro name="drive_wheel" params="*origin parent suffix drive_vel:=^|100 steer_vel:=^|100"> -->
+  <xacro:macro name="drive_wheel" params="*origin parent suffix">
     <xacro:cob_caster_hub parent="${parent}" suffix="${suffix}_caster" >
       <xacro:insert_block name="origin" />

File: raw_description/urdf/base_long/base.urdf.xacro (robot description, xacro)
@@ -5,4 +5,7 @@
   <!-- drive_wheel module -->
   <xacro:include filename="$(find cob_description)/urdf/drive_wheel/drive_wheel.urdf.xacro" />
+  <!-- sensors -->
+  <xacro:include filename="$(find cob_description)/urdf/sensors/sick_s300_laser.urdf.xacro"/>
+  <xacro:include filename="$(find cob_description)/urdf/sensors/kinect.urdf.xacro"/>
   <!-- properties -->
   <xacro:property name="caster_offset_x" value="0.368" />  <!--modify here-->
@@ -59,7 +62,13 @@
     </joint>
     <link name="${name}_link">
-      <xacro:box_inertial x="1.04" y="0.58" z="0.12" mass="${base_mass}">
+      <inertial>
+        <origin xyz="0 0 0" />
+        <mass value="${base_mass}" />
+        <inertia ixx="9.64" ixy="-0.02" ixz="0.44"
+                 iyy="11.33" iyz="-0.007" izz="3.07" />
+      </inertial>
+      <!-- <xacro:box_inertial x="1.04" y="0.58" z="0.12" mass="${base_mass}">
         <origin xyz="0 0 0" rpy="0 0 0"/>
-      </xacro:box_inertial>
+      </xacro:box_inertial> -->
       <visual>
         <origin xyz="0 0 0.209" rpy="0 0 0" />
@@ -89,4 +98,16 @@
       <origin xyz="${-caster_offset_x} ${caster_offset_y_br} ${caster_offset_z}" rpy="0 0 0" />
     </xacro:drive_wheel>
+    <!-- base laser front -->
+    <xacro:sick_s300_laser_v0 name="${name}_laser_front" parent="${name}">
+      <origin xyz="${laser_front_x} ${laser_front_y} ${laser_front_z}" rpy="${laser_front_roll} ${laser_front_pitch} ${laser_front_yaw}" />
+    </xacro:sick_s300_laser_v0>
+    <!-- base laser rear -->
+    <xacro:sick_s300_laser_v0 name="${name}_laser_rear" parent="${name}">
+      <origin xyz="${laser_rear_x} ${laser_rear_y} ${laser_rear_z}" rpy="${laser_rear_roll} ${laser_rear_pitch} ${laser_rear_yaw}" />
+    </xacro:sick_s300_laser_v0>
+    <!-- cam3d -->
+    <!--xacro:cob_kinect_v0 name="${name}_cam3d" ros_topic="cam3d" parent="${name}_link">
+      <origin xyz="0.51 0.12 0.27" rpy="-${M_PI/2} 0 -${M_PI/2}" />
+    </xacro:cob_kinect_v0-->
     <!-- battery front-->
     <xacro:cob_batteries name="${name}_battery_front" parent="${name}_link">

File: raw_description/urdf/base_short/base.urdf.xacro (robot description, xacro)
@@ -5,4 +5,7 @@
   <!-- drive_wheel module -->
   <xacro:include filename="$(find cob_description)/urdf/drive_wheel/drive_wheel.urdf.xacro" />
+  <!-- sensors -->
+  <xacro:include filename="$(find cob_description)/urdf/sensors/sick_s300_laser.urdf.xacro"/>
+  <xacro:include filename="$(find cob_description)/urdf/sensors/kinect.urdf.xacro"/>
   <!-- properties -->
   <xacro:property name="caster_offset_x" value="0.228" />  <!--modify here-->
@@ -93,4 +96,16 @@
       <origin xyz="${-caster_offset_x} ${caster_offset_y_br} ${caster_offset_z}" rpy="0 0 0" />
     </xacro:drive_wheel>
+    <!-- base laser front -->
+    <xacro:sick_s300_laser_v0 name="${name}_laser_front" parent="${name}">
+      <origin xyz="${laser_front_x} ${laser_front_y} ${laser_front_z}" rpy="${laser_front_roll} ${laser_front_pitch} ${laser_front_yaw}" />
+    </xacro:sick_s300_laser_v0>
+    <!-- base laser rear -->
+    <xacro:sick_s300_laser_v0 name="${name}_laser_rear" parent="${name}">
+      <origin xyz="${laser_rear_x} ${laser_rear_y} ${laser_rear_z}" rpy="${laser_rear_roll} ${laser_rear_pitch} ${laser_rear_yaw}" />
+    </xacro:sick_s300_laser_v0>
+    <!-- cam3d -->
+    <!--xacro:cob_kinect_v0 name="${name}_cam3d" ros_topic="cam3d" parent="${name}_link">
+      <origin xyz="0.51 0.12 0.27" rpy="-${M_PI/2} 0 -${M_PI/2}" />
+    </xacro:cob_kinect_v0-->
     <!-- battery-->
     <xacro:cob_batteries name="${name}_battery" parent="${name}_link">
