Commit message: add sr300 on the base facing right

File: cob_description/urdf/sensors/realsense_brad.gazebo.xacro (robot description, xacro)
@@ -2,10 +2,8 @@
 <robot xmlns:xacro="http://www.ros.org/wiki/xacro">
   <!-- use default values of realsense_camera/r200_nodelet_rgbd -->
-  <xacro:macro name="realsense_rgb_gazebo_v0" params="link_name
-                                               frame_name
-                                               camera_name
+  <xacro:macro name="realsense_gazebo" params="name ros_topic
                                                depth_fps:=30.0 depth_height:=360 depth_width:=480
                                                color_fps:=30.0 color_height:=480 color_width:=640" >
-    <gazebo reference="${link_name}">
+    <gazebo reference="${name}_link">
       <sensor type="depth" name="${name}_depth_frame">
         <always_on>true</always_on>
@@ -28,13 +26,13 @@
           </noise>
         </camera>
-        <plugin name="${link_name}_controller" filename="libgazebo_ros_openni_kinect.so">
+        <plugin name="${name}_frame_controller" filename="libgazebo_ros_openni_kinect.so">
           <updateRate>${color_fps}</updateRate>
-          <cameraName>${camera_name}_rgb</cameraName>
-          <frameName>${frame_name}</frameName>
-          <imageTopicName>/${camera_name}/rgb/image_raw</imageTopicName>
-          <cameraInfoTopicName>/${camera_name}/rgb/camera_info</cameraInfoTopicName>
-          <pointCloudTopicName>/${camera_name}/depth_registered/points</pointCloudTopicName>
-          <depthImageTopicName>/${camera_name}/depth_registered/image_raw</depthImageTopicName>
-          <depthImageCameraInfoTopicName>/${camera_name}/depth_registered/camera_info</depthImageCameraInfoTopicName>
+          <cameraName>${ros_topic}</cameraName>
+          <frameName>${name}_rgb_optical_frame</frameName>
+          <imageTopicName>rgb/image_raw</imageTopicName>
+          <cameraInfoTopicName>rgb/camera_info</cameraInfoTopicName>
+          <pointCloudTopicName>depth_registered/points</pointCloudTopicName>
+          <depthImageTopicName>depth_registered/image_raw</depthImageTopicName>
+          <depthImageCameraInfoTopicName>depth_registered/camera_info</depthImageCameraInfoTopicName>
           <pointCloudCutoff>0.5</pointCloudCutoff>
           <pointCloudCutoffMax>5.0</pointCloudCutoffMax>
@@ -50,5 +48,5 @@
         </plugin>
       </sensor>
-      <material value="Gazebo/Red" />
+      <material>IPA/LightGrey</material>
     </gazebo>
   </xacro:macro>

File: cob_description/urdf/sensors/realsense_brad.urdf.xacro (robot description, xacro)
@@ -3,11 +3,10 @@
   <xacro:include filename="$(find cob_description)/urdf/sensors/realsense.gazebo.xacro" />
   <xacro:macro name="realsense" params="name parent ros_topic *origin">
-    <!-- realsense rgb sensor physical attachment -->
-    <joint name="${name}_realsense_rgb_joint" type="fixed">
+    <joint name="${name}_joint" type="fixed">
       <xacro:insert_block name="origin" />
       <parent link="${parent}"/>
-      <child link="${name}_realsense_rgb_link"/>
+      <child link="${name}_link"/>
     </joint>
-    <link name="${name}_realsense_rgb_link" >
+    <link name="${name}_link">
       <inertial>
         <mass value="0.564" />
@@ -29,13 +28,6 @@
       </collision>
     </link>
-    <!-- realsense rgb sensor frame -->
-    <joint name="${name}_realsense_rgb_optical_frame_joint" type="fixed">
-      <origin xyz="0.0 0.0 0.0" rpy="0.0 0.0 0.0" />
-      <parent link="${name}_realsense_rgb_link"/>
-      <child link="${name}_realsense_rgb_optical_frame"/>
-    </joint>
-    <link name="${name}_realsense_rgb_optical_frame"/>
-    <!-- gazebo extensions -->
-    <xacro:realsense_rgb_gazebo_v0 link_name="${name}_realsense_rgb_link" frame_name="${name}_realsense_rgb_optical_frame" camera_name="${name}"/>
+    <!-- extensions -->
+    <xacro:realsense_gazebo name="${name}" ros_topic="${ros_topic}" />
   </xacro:macro>
 </robot>
