Commit message: the bug = camera view simulated in gazebo was upside down! The reason was that the dae was mirrored. i use blender to fix the dae, then the view of the camera becomes correct.

File: cob_description/urdf/sensors/realsense.gazebo.xacro (robot description, xacro)
@@ -51,5 +51,4 @@
         </plugin>
       </sensor>
-      <material value="Gazebo/Red" />
     </gazebo>
   </xacro:macro>

File: cob_description/urdf/sensors/realsense.urdf.xacro (robot description, xacro)
@@ -45,5 +45,7 @@
       <child link="${name}_realsense_rgb_optical_frame"/>
     </joint>
-    <link name="${name}_realsense_rgb_optical_frame"/>
+    <link name="${name}_realsense_rgb_optical_frame">
+      <origin xyz="0.0 0.0 0.0" rpy="0.0 0.0 0.0" />
+    </link>
     <!-- gazebo extensions -->
     <xacro:realsense_rgb_gazebo_v0 link_name="${name}_realsense_rgb_link" frame_name="${name}_realsense_rgb_optical_frame" camera_name="${name}"/>

Commit message: add sim-sr300

File: cob_description/urdf/sensors/realsense.gazebo.xacro (robot description, xacro)
@@ -3,5 +3,7 @@
 <!-- https://github.com/PR2/pr2_common/blob/kinetic-devel/pr2_description/urdf/sensors/kinect2.gazebo.xacro -->
   <!-- use default values of realsense_camera/r200_nodelet_rgbd -->
-  <xacro:macro name="realsense_rgb_gazebo_v0" params="link_name
+  <xacro:macro name="realsense_rgb_gazebo_v0" params="
+                                               name
+                                               link_name
                                                frame_name
                                                camera_name

File: cob_description/urdf/sensors/realsense.urdf.xacro (robot description, xacro)
@@ -2,6 +2,13 @@
 <robot xmlns:xacro="http://www.ros.org/wiki/xacro">
 <!-- https://github.com/PR2/pr2_common/blob/kinetic-devel/pr2_description/urdf/sensors/kinect2.urdf.xacro -->
-  <xacro:include filename="$(find cob_description)/urdf/sensors/realsense.gazebo.xacro" />
-  <xacro:macro name="realsense" params="name parent ros_topic *origin">
+  <!-- <xacro:include filename="$(find cob_description)/urdf/sensors/realsense.gazebo.xacro" /> -->
+  <xacro:macro name="realsense" params="sim name parent ros_topic *origin">
+    <!-- The rpy for simulation is different from the rpy setup for the actual camera. If we use the rpy from actual camera in simulation, the view will be wrong -->
+    <xacro:if value="${sim}">
+      <xacro:property name="realsense_rgb_link_visual_rpy" value="${-90/180*pi} 0.0 ${-90/180*pi}"/>
+    </xacro:if>
+    <xacro:unless value="${sim}">
+      <xacro:property name="realsense_rgb_link_visual_rpy" value="0.0 0.0 0.0"/>
+    </xacro:unless>
     <!-- realsense rgb sensor physical attachment -->
     <joint name="${name}_realsense_rgb_joint" type="fixed">
@@ -17,8 +24,8 @@
       </inertial>
       <visual>
-       <origin xyz="0 0 0" rpy="0 0 0"/>
+       <origin xyz="0 0 0" rpy="${realsense_rgb_link_visual_rpy}"/>
         <geometry>
           <!--<box size="0.002 0.002 0.002"/>-->
-          <mesh filename="package://cob_description/meshes/sensors/sr300_optical_link.dae"/>
+          <mesh filename="package://cob_description/meshes/sensors/untitled.dae"/>
           <!-- <mesh filename="package://cob_description/meshes/sensors/sr300_optical_link.STL"/> -->
           <!-- <mesh filename="package://cob_description/urdf/sensors/intel_realsense_r200/meshes/realsense_r200.dae"/> -->
@@ -49,5 +56,5 @@
     </link>
     <!-- gazebo extensions -->
-    <!-- <xacro:realsense_rgb_gazebo_v0 link_name="${name}_realsense_rgb_link" frame_name="${name}_realsense_rgb_optical_frame" camera_name="${name}"/> -->
+    <!-- <xacro:realsense_rgb_gazebo_v0 name="${name}" link_name="${name}_realsense_rgb_link" frame_name="${name}_realsense_rgb_optical_frame" camera_name="${name}_gazebo"/> -->
   </xacro:macro>
 </robot>

Commit message: add options for visualize_wrist_sr300_simulator and visualize_sick_s300_simulator

File: cob_description/urdf/sensors/realsense.gazebo.xacro (robot description, xacro)
@@ -8,9 +8,31 @@
                                                frame_name
                                                camera_name
+                                               visualize_wrist_sr300_simulator
                                                depth_fps:=30.0 depth_height:=360 depth_width:=480
                                                color_fps:=30.0 color_height:=480 color_width:=640" >
     <gazebo reference="${link_name}">
+      <!-- This is used for visualize the rgb in gazebo -->
+      <!-- this camera sensor setup is copied from pr2 model in .gazebo/models/pr2/model.sdf -->
+      <!-- https://bitbucket.org/osrf/gazebo_models/src/220aa60a2eaa5f31b52429d08c8e94bd05646e23/pr2/model.sdf?at=default&fileviewer=file-view-default -->
+      <sensor name="${name}_rgb_frame" type="camera">
+        <always_on>true</always_on>
+        <visualize>${visualize_wrist_sr300_simulator}</visualize>
+        <update_rate>${color_fps}</update_rate>
+        <camera>
+          <horizontal_fov>${74.0*M_PI/180.0}</horizontal_fov>
+          <image>
+            <width>${color_width}</width>
+            <height>${color_height}</height>
+            <format>R8G8B8</format>
+          </image>
+          <clip>
+            <near>0.15</near>
+            <far>1.0</far>
+          </clip>
+        </camera>
+      </sensor>
       <sensor type="depth" name="${name}_depth_frame">
         <always_on>true</always_on>
+        <visualize>true</visualize>
         <update_rate>${color_fps}</update_rate>
         <camera>

File: cob_description/urdf/sensors/sick_s300_laser.gazebo.xacro (robot description, xacro)
@@ -1,11 +1,13 @@
 <?xml version="1.0"?>
 <robot xmlns:xacro="http://www.ros.org/wiki/xacro">
-  <xacro:macro name="sick_s300_laser_gazebo_v0" params="name">
+  <xacro:macro name="sick_s300_laser_gazebo_v0" params="visualize_sick_s300_simulator name">
     <gazebo reference="${name}_link">
+      <!-- this ray sensor setup is similar to the one in pr2 model in .gazebo/models/pr2/model.sdf -->
+      <!-- https://bitbucket.org/osrf/gazebo_models/src/220aa60a2eaa5f31b52429d08c8e94bd05646e23/pr2/model.sdf?at=default&fileviewer=file-view-default -->
       <sensor name="${name}" type="ray">
         <always_on>true</always_on>
+        <visualize>${visualize_sick_s300_simulator}</visualize>
         <update_rate>12.0</update_rate>
         <pose>0 0 0 0 0 0</pose>
-        <visualize>false</visualize>
         <ray>
           <scan>

File: cob_description/urdf/sensors/sick_s300_laser.urdf.xacro (robot description, xacro)
@@ -4,5 +4,5 @@
   <xacro:property name="cylinder_radius" value="0.05" />  <!--simple collision model for the laser -->
   <xacro:property name="cylinder_length" value="0.15" />
-  <xacro:macro name="sick_s300_laser_v0" params="name parent *origin">
+  <xacro:macro name="sick_s300_laser_v0" params="visualize_sick_s300_simulator sim name parent *origin">
     <joint name="${name}_joint" type="fixed">
       <axis xyz="0 1 0" />
@@ -31,5 +31,7 @@
     </link>
     <!-- gazebo extensions -->
-    <xacro:sick_s300_laser_gazebo_v0 name="${name}"/>
+    <xacro:if value="${sim}">
+      <xacro:sick_s300_laser_gazebo_v0 visualize_sick_s300_simulator="${visualize_sick_s300_simulator}" name="${name}"/>
+    </xacro:if>
   </xacro:macro>
 </robot>

File: raw_description/urdf/base_long/base.urdf.xacro (robot description, xacro)
@@ -26,5 +26,5 @@
   <xacro:property name="battery_size_z" value="0.26" />
   <!-- battery macros-->
-  <xacro:macro name="cob_batteries" params="name parent *origin ">
+  <xacro:macro name="cob_batteries" params="sim name parent *origin ">
     <joint name="${name}_battery_joint" type="fixed">
       <xacro:insert_block name="origin" />
@@ -52,7 +52,9 @@
     </link>
     <!-- extensions -->
-    <xacro:batteries_gazebo name="${name}" />
+    <xacro:if value="${sim}">
+      <xacro:batteries_gazebo name="${name}" />
+    </xacro:if>
   </xacro:macro>
-  <xacro:macro name="raw_base" params="name">
+  <xacro:macro name="raw_base" params="sim visualize_sick_s300_simulator name">
     <link name="${name}_footprint"/>
     <joint name="${name}_footprint_joint" type="fixed">
@@ -99,9 +101,9 @@
     </xacro:drive_wheel>
     <!-- base laser front -->
-    <xacro:sick_s300_laser_v0 name="${name}_laser_front" parent="${name}">
+    <xacro:sick_s300_laser_v0 visualize_sick_s300_simulator="${visualize_sick_s300_simulator}" sim="${sim}" name="${name}_laser_front" parent="${name}">
       <origin xyz="${laser_front_x} ${laser_front_y} ${laser_front_z}" rpy="${laser_front_roll} ${laser_front_pitch} ${laser_front_yaw}" />
     </xacro:sick_s300_laser_v0>
     <!-- base laser rear -->
-    <xacro:sick_s300_laser_v0 name="${name}_laser_rear" parent="${name}">
+    <xacro:sick_s300_laser_v0 visualize_sick_s300_simulator="${visualize_sick_s300_simulator}" sim="${sim}" name="${name}_laser_rear" parent="${name}">
       <origin xyz="${laser_rear_x} ${laser_rear_y} ${laser_rear_z}" rpy="${laser_rear_roll} ${laser_rear_pitch} ${laser_rear_yaw}" />
     </xacro:sick_s300_laser_v0>
@@ -111,13 +113,15 @@
     </xacro:cob_kinect_v0-->
     <!-- battery front-->
-    <xacro:cob_batteries name="${name}_battery_front" parent="${name}_link">
+    <xacro:cob_batteries sim="${sim}" name="${name}_battery_front" parent="${name}_link">
       <origin xyz="${-battery_offset_x_f} ${battery_offset_y_f} ${battery_offset_z}" rpy="${M_PI/2} 0 ${-M_PI/2}" />
     </xacro:cob_batteries>
     <!-- battery rear-->
-    <xacro:cob_batteries name="${name}_battery_rear" parent="${name}_link">
+    <xacro:cob_batteries sim="${sim}" name="${name}_battery_rear" parent="${name}_link">
       <origin xyz="${battery_offset_x_r} ${battery_offset_y_r} ${battery_offset_z}" rpy="${M_PI/2} 0 ${-M_PI/2}" />
     </xacro:cob_batteries>
     <!-- gazebo extensions -->
-    <xacro:base_gazebo name="${name}" />
+    <xacro:if value="${sim}">
+      <xacro:base_gazebo name="${name}" />
+    </xacro:if>
     <!-- ros_control plugin -->
     <gazebo>

Commit message: both gazebo and real cameras working

File: cob_description/urdf/sensors/realsense.gazebo.xacro (robot description, xacro)
@@ -4,16 +4,16 @@
   <!-- use default values of realsense_camera/r200_nodelet_rgbd -->
   <xacro:macro name="realsense_rgb_gazebo_v0" params="
-                                               name
-                                               link_name
-                                               frame_name
-                                               camera_name
-                                               visualize_wrist_sr300_simulator
-                                               depth_fps:=30.0 depth_height:=360 depth_width:=480
-                                               color_fps:=30.0 color_height:=480 color_width:=640" >
+    name link_name frame_name camera_name visualize_wrist_sr300_simulator
+    depth_fps:=30.0
+    depth_height:=360
+    depth_width:=480
+    color_fps:=30.0
+    color_height:=480
+    color_width:=640" >
     <gazebo reference="${link_name}">
-      <!-- This is used for visualize the rgb in gazebo -->
       <!-- this camera sensor setup is copied from pr2 model in .gazebo/models/pr2/model.sdf -->
       <!-- https://bitbucket.org/osrf/gazebo_models/src/220aa60a2eaa5f31b52429d08c8e94bd05646e23/pr2/model.sdf?at=default&fileviewer=file-view-default -->
-      <sensor name="${name}_rgb_frame" type="camera">
+      <!-- just for visualization in gazebo -->
+      <sensor name="${name}_rgb_visualizer" type="camera">
         <always_on>true</always_on>
         <visualize>${visualize_wrist_sr300_simulator}</visualize>
@@ -27,12 +27,62 @@
           </image>
           <clip>
-            <near>0.15</near>
-            <far>1.0</far>
+            <near>0.2</near>
+            <far>1.5</far>
           </clip>
         </camera>
       </sensor>
-      <sensor type="depth" name="${name}_depth_frame">
+      <!-- https://github.com/PR2/pr2_common/blob/kinetic-devel/pr2_description/urdf/sensors/kinect2.gazebo.xacro -->
+      <sensor name="${name}_rgb_gazebo_simulation" type="depth">
         <always_on>true</always_on>
-        <visualize>true</visualize>
+        <update_rate>${color_fps}</update_rate>
+        <camera>
+          <horizontal_fov>${74.0*M_PI/180.0}</horizontal_fov>
+          <image>
+            <width>${color_width}</width>
+            <height>${color_height}</height>
+            <format>R8G8B8</format>
+          </image>
+          <clip>
+            <near>0.2</near>
+            <far>1.5</far>
+          </clip>
+        </camera>
+        <plugin name="${name}_rgb_gazebo_simulation_controller" filename="libgazebo_ros_openni_kinect.so">
+          <alwaysOn>true</alwaysOn>
+          <updateRate>${color_fps}</updateRate>
+          <cameraName>${camera_name}_rgb_gazebo_simulation</cameraName>
+          <frameName>${frame_name}</frameName>
+          <imageTopicName>/${camera_name}/rgb/image_raw</imageTopicName>
+          <cameraInfoTopicName>/${camera_name}/rgb/camera_info</cameraInfoTopicName>
+          <depthImageTopicName>/${camera_name}/depth/image_raw</depthImageTopicName>
+          <depthImageCameraInfoTopicName>/${camera_name}/depth/camera_info</depthImageCameraInfoTopicName>
+          <pointCloudTopicName>/${camera_name}/depth_registered/points</pointCloudTopicName>
+          <pointCloudCutoff>0.5</pointCloudCutoff>
+          <pointCloudCutoffMax>5.0</pointCloudCutoffMax>
+          <distortionK1>0.0</distortionK1>
+          <distortionK2>0.0</distortionK2>
+          <distortionK3>0.0</distortionK3>
+          <distortionT1>0.0</distortionT1>
+          <distortionT2>0.0</distortionT2>
+          <CxPrime>0.0</CxPrime>
+          <Cx>0.0</Cx>
+          <Cy>0.0</Cy>
+          <focalLength>0.0</focalLength>
+        </plugin>
+      </sensor>
+    </gazebo>
+  </xacro:macro>
+  <!-- https://github.com/PR2/pr2_common/blob/kinetic-devel/pr2_description/urdf/sensors/kinect2.gazebo.xacro -->
+  <xacro:macro name="realsense_ir_gazebo_v0" params="
+    name link_name frame_name camera_name visualize_wrist_sr300_simulator
+    depth_fps:=30.0
+    depth_height:=360
+    depth_width:=480
+    color_fps:=30.0
+    color_height:=480
+    color_width:=640" >
+    <gazebo reference="${link_name}">
+      <sensor type="depth" name="${name}_ir_gazebo_simulation">
+        <always_on>true</always_on>
         <update_rate>${color_fps}</update_rate>
         <camera>
@@ -44,6 +94,8 @@
           </image>
           <clip>
-            <near>0.15</near>
-            <far>1.0</far>
+            <!-- <near>0.15</near> -->
+            <!-- <far>1.0</far> -->
+            <near>0.2</near>
+            <far>1.5</far>
           </clip>
           <noise>
@@ -53,13 +105,14 @@
           </noise>
         </camera>
-        <plugin name="${link_name}_controller" filename="libgazebo_ros_openni_kinect.so">
+        <plugin name="${name}_ir_gazebo_simulation_controller" filename="libgazebo_ros_openni_kinect.so">
+          <alwaysOn>true</alwaysOn>
           <updateRate>${color_fps}</updateRate>
-          <cameraName>${camera_name}_rgb</cameraName>
+          <cameraName>${camera_name}_ir_gazebo_simulation</cameraName>
           <frameName>${frame_name}</frameName>
-          <imageTopicName>/${camera_name}/rgb/image_raw</imageTopicName>
-          <cameraInfoTopicName>/${camera_name}/rgb/camera_info</cameraInfoTopicName>
-          <pointCloudTopicName>/${camera_name}/depth_registered/points</pointCloudTopicName>
-          <depthImageTopicName>/${camera_name}/depth_registered/image_raw</depthImageTopicName>
-          <depthImageCameraInfoTopicName>/${camera_name}/depth_registered/camera_info</depthImageCameraInfoTopicName>
+          <imageTopicName>/${camera_name}/ir/image_raw</imageTopicName>
+          <cameraInfoTopicName>/${camera_name}/ir/camera_info</cameraInfoTopicName>
+          <depthImageTopicName>/${camera_name}/depth/image_raw</depthImageTopicName>
+          <depthImageCameraInfoTopicName>/${camera_name}/depth/camera_info</depthImageCameraInfoTopicName>
+          <pointCloudTopicName>/${camera_name}/depth/points</pointCloudTopicName>
           <pointCloudCutoff>0.5</pointCloudCutoff>
           <pointCloudCutoffMax>5.0</pointCloudCutoffMax>

File: cob_description/urdf/sensors/realsense.urdf.xacro (robot description, xacro)
@@ -2,27 +2,30 @@
 <robot xmlns:xacro="http://www.ros.org/wiki/xacro">
 <!-- https://github.com/PR2/pr2_common/blob/kinetic-devel/pr2_description/urdf/sensors/kinect2.urdf.xacro -->
-  <!-- <xacro:include filename="$(find cob_description)/urdf/sensors/realsense.gazebo.xacro" /> -->
-  <xacro:macro name="realsense" params="sim name parent ros_topic *origin">
-    <!-- The rpy for simulation is different from the rpy setup for the actual camera. If we use the rpy from actual camera in simulation, the view will be wrong -->
+  <xacro:macro name="realsense" params="sim name parent *origin">
+    <!-- The origin roll pitch yaw for the frame_joints in gazebo simulation is different from the one for the real camera! -->
     <xacro:if value="${sim}">
-      <xacro:property name="realsense_rgb_link_visual_rpy" value="${-90/180*pi} 0.0 ${-90/180*pi}"/>
+      <!-- this is for pointing the camera to the right direction in gazebo -->
+      <xacro:property name="frame_joint_rpy" value="0.0 ${-90/180*pi} ${90/180*pi}"/>
+      <!-- this is for placing the point cloud on the right position with the correct transformation from the robot in rviz -->
+      <xacro:property name="optical_frame_joint_rpy" value="${-90/180*pi} 0.0 ${-90/180*pi}"/>
     </xacro:if>
     <xacro:unless value="${sim}">
-      <xacro:property name="realsense_rgb_link_visual_rpy" value="0.0 0.0 0.0"/>
+      <xacro:property name="frame_joint_rpy" value="0.0 0.0 0.0"/>
+      <xacro:property name="optical_frame_joint_rpy" value="0.0 0.0 0.0"/>
     </xacro:unless>
-    <!-- realsense rgb sensor physical attachment -->
-    <joint name="${name}_realsense_rgb_joint" type="fixed">
+    <!-- camera physical attachment -->
+    <joint name="${name}_joint" type="fixed">
       <xacro:insert_block name="origin" />
       <parent link="${parent}"/>
-      <child link="${name}_realsense_rgb_link"/>
+      <child link="${name}_link"/>
     </joint>
-    <link name="${name}_realsense_rgb_link" >
+    <link name="${name}_link" >
       <inertial>
         <mass value="0.564" />
-        <origin xyz="0 0 0" />
+        <origin xyz="0.0 0.0 0.0" rpy="0.0 0.0 0.0" />
         <inertia ixx="0.003881243" ixy="0.0" ixz="0.0" iyy="0.000498940" iyz="0.0" izz="0.003879257" />
       </inertial>
       <visual>
-       <origin xyz="0 0 0" rpy="${realsense_rgb_link_visual_rpy}"/>
+       <origin xyz="0.0 0.0 0.0" rpy="0.0 0.0 0.0"/>
         <geometry>
           <!--<box size="0.002 0.002 0.002"/>-->
@@ -31,12 +34,12 @@
           <!-- <mesh filename="package://cob_description/urdf/sensors/intel_realsense_r200/meshes/realsense_r200.dae"/> -->
         </geometry>
-        <material name="sr300_gray">
-          <color rgba="0.75 0.75 0.75 1" />
+        <!-- <material name="sr300_gray"> -->
+          <!-- <color rgba="0.75 0.75 0.75 1" /> -->
           <!-- <color rgba="0.1 0.1 0.1 1" /> -->
           <!--<color rgba="0.2 0.2 1 1" />-->
-        </material>
+        <!-- </material> -->
       </visual>
       <collision>
-        <origin xyz="-0.025 0.0 -0.01" rpy="0 0 0"/>
+        <origin xyz="-0.025 0.0 -0.01" rpy="0.0 0.0 0.0"/>
         <geometry>
           <!-- <box size="0.007 0.130 0.0118"/> -->
@@ -46,15 +49,58 @@
       </collision>
     </link>
-    <!-- realsense rgb sensor frame -->
-    <joint name="${name}_realsense_rgb_optical_frame_joint" type="fixed">
-      <origin xyz="0.0 0.0 0.0" rpy="0.0 0.0 0.0" />
-      <parent link="${name}_realsense_rgb_link"/>
-      <child link="${name}_realsense_rgb_optical_frame"/>
+    <!-- 1(1) rgb_frame -->
+    <joint name="${name}_rgb_frame_joint" type="fixed">
+      <origin xyz="0.0 0.0 0.0" rpy="${frame_joint_rpy}" />
+      <parent link="${name}_link"/>
+      <child link="${name}_rgb_frame"/>
     </joint>
-    <link name="${name}_realsense_rgb_optical_frame">
+    <link name="${name}_rgb_frame">
       <origin xyz="0.0 0.0 0.0" rpy="0.0 0.0 0.0" />
     </link>
-    <!-- gazebo extensions -->
-    <!-- <xacro:realsense_rgb_gazebo_v0 name="${name}" link_name="${name}_realsense_rgb_link" frame_name="${name}_realsense_rgb_optical_frame" camera_name="${name}_gazebo"/> -->
+    <!-- 1(2) rgb_optical_frame -->
+    <joint name="${name}_rgb_optical_frame_joint" type="fixed">
+      <origin xyz="0.0 0.0 0.0" rpy="${optical_frame_joint_rpy}" />
+      <parent link="${name}_rgb_frame"/>
+      <child link="${name}_rgb_optical_frame"/>
+    </joint>
+    <link name="${name}_rgb_optical_frame">
+      <origin xyz="0.0 0.0 0.0" rpy="0.0 0.0 0.0" />
+    </link>
+    <!-- 2(1) depth_frame -->
+    <joint name="${name}_depth_frame_joint" type="fixed">
+      <origin xyz="0.0 0.0 0.0" rpy="${frame_joint_rpy}" />
+      <parent link="${name}_link"/>
+      <child link="${name}_depth_frame"/>
+    </joint>
+    <link name="${name}_depth_frame">
+      <origin xyz="0.0 0.0 0.0" rpy="0.0 0.0 0.0" />
+    </link>
+    <!-- 2(2) depth_optical_frame -->
+    <joint name="${name}_depth_optical_frame_joint" type="fixed">
+      <origin xyz="0.0 0.0 0.0" rpy="${optical_frame_joint_rpy}" />
+      <parent link="${name}_depth_frame"/>
+      <child link="${name}_depth_optical_frame"/>
+    </joint>
+    <link name="${name}_depth_optical_frame">
+      <origin xyz="0.0 0.0 0.0" rpy="0.0 0.0 0.0" />
+    </link>
+    <!-- 3(1) ir_frame -->
+    <joint name="${name}_ir_frame_joint" type="fixed">
+      <origin xyz="0.0 0.0 0.0" rpy="${frame_joint_rpy}" />
+      <parent link="${name}_link"/>
+      <child link="${name}_ir_frame"/>
+    </joint>
+    <link name="${name}_ir_frame">
+      <origin xyz="0.0 0.0 0.0" rpy="0.0 0.0 0.0" />
+    </link>
+    <!-- 3(2) ir_optical_frame -->
+    <joint name="${name}_ir_optical_frame_joint" type="fixed">
+      <origin xyz="0.0 0.0 0.0" rpy="${optical_frame_joint_rpy}" />
+      <parent link="${name}_ir_frame"/>
+      <child link="${name}_ir_optical_frame"/>
+    </joint>
+    <link name="${name}_ir_optical_frame">
+      <origin xyz="0.0 0.0 0.0" rpy="0.0 0.0 0.0" />
+    </link>
   </xacro:macro>
 </robot>
