Commit message: fix bug

File: cob_description/urdf/sensors/r200.urdf.xacro (robot description, xacro)
@@ -15,4 +15,5 @@
     </xacro:if>
     <xacro:unless value="${sim}">
+      <xacro:property name="frame_joint_xyz" value="0.0 0.0 0.0"/>
       <xacro:property name="frame_joint_rpy" value="0.0 0.0 0.0"/>
       <xacro:property name="optical_frame_joint_rpy" value="0.0 0.0 0.0"/>

Commit message: fix real r200 setting

File: cob_description/urdf/sensors/r200.urdf.xacro (robot description, xacro)
@@ -17,5 +17,5 @@
       <xacro:property name="frame_joint_xyz" value="0.0 0.0 0.0"/>
       <xacro:property name="frame_joint_rpy" value="0.0 0.0 0.0"/>
-      <xacro:property name="optical_frame_joint_rpy" value="0.0 0.0 0.0"/>
+      <xacro:property name="optical_frame_joint_rpy" value="0.0 0.0 ${90/180*pi}"/>
     </xacro:unless>
     <!-- camera physical attachment -->

Commit message: update bug for real robot frame joint xyz

File: cob_description/urdf/sensors/r200.urdf.xacro (robot description, xacro)
@@ -15,5 +15,5 @@
     </xacro:if>
     <xacro:unless value="${sim}">
-      <xacro:property name="frame_joint_xyz" value="0.0 0.0 0.0"/>
+      <xacro:property name="frame_joint_xyz" value="0.0 0.047625 0.0111"/>
       <xacro:property name="frame_joint_rpy" value="0.0 0.0 0.0"/>
       <xacro:property name="optical_frame_joint_rpy" value="0.0 0.0 ${90/180*pi}"/>
