Commit message: fix transformation bw r200 and palm, lens and r200 via compute-obj2obj in yuripy, refactor realsense -> r200

File: cob_description/urdf/sensors/r200.gazebo.xacro (robot description, xacro)
@@ -3,5 +3,5 @@
 <!-- https://github.com/PR2/pr2_common/blob/kinetic-devel/pr2_description/urdf/sensors/kinect2.gazebo.xacro -->
   <!-- use default values of realsense_camera/r200_nodelet_rgbd -->
-  <xacro:macro name="realsense_rgb_gazebo_v0" params="
+  <xacro:macro name="r200_rgb_gazebo_v0" params="
     name link_name frame_name camera_name visualize_wrist_camera_simulator
     depth_fps:=30.0
@@ -76,5 +76,5 @@
   </xacro:macro>
   <!-- https://github.com/PR2/pr2_common/blob/kinetic-devel/pr2_description/urdf/sensors/kinect2.gazebo.xacro -->
-  <xacro:macro name="realsense_ir_gazebo_v0" params="
+  <xacro:macro name="r200_ir_gazebo_v0" params="
     name link_name frame_name camera_name visualize_wrist_camera_simulator
     depth_fps:=30.0

File: cob_description/urdf/sensors/r200.urdf.xacro (robot description, xacro)
@@ -2,10 +2,14 @@
 <robot xmlns:xacro="http://www.ros.org/wiki/xacro">
 <!-- https://github.com/PR2/pr2_common/blob/kinetic-devel/pr2_description/urdf/sensors/kinect2.urdf.xacro -->
-  <xacro:macro name="realsense" params="sim name parent *origin">
+  <xacro:macro name="r200" params="sim name parent *origin">
     <!-- The origin roll pitch yaw for the frame_joints in gazebo simulation is different from the one for the real camera! -->
     <xacro:if value="${sim}">
       <!-- this is for pointing the camera to the right direction in gazebo -->
-      <xacro:property name="frame_joint_rpy" value="0.0 ${-90/180*pi} ${90/180*pi}"/>
+      <!-- XXX: Visualizing camera view in gazebo will help you verify the exact position of that camera lens in relative to the physical camera "cube" -->
+      <!-- frame_joint_xyz and frame_joint_rpy = lens_in_r200_mat -->
+      <xacro:property name="frame_joint_xyz" value="0.0 0.047625 0.0111"/>
+      <xacro:property name="frame_joint_rpy" value="0.0 ${-90/180*pi} ${180/180*pi}"/>
       <!-- this is for placing the point cloud on the right position with the correct transformation from the robot in rviz -->
+      <!-- XXX: Visualizing camera view in rviz will help you verify the camera visual image transformation (inverted or not, tilted or not ...) -->
       <xacro:property name="optical_frame_joint_rpy" value="${-90/180*pi} 0.0 ${-90/180*pi}"/>
     </xacro:if>
@@ -29,5 +33,5 @@
        <origin xyz="0.0 0.0 0.0" rpy="0.0 0.0 0.0"/>
         <geometry>
-          <box size="0.02 0.02 0.02"/>
+          <box size="0.01905 0.1335 0.0222"/>
           <!-- <mesh filename="package://cob_description/meshes/sensors/sr300_optical_link.dae"/> -->
         </geometry>
@@ -39,7 +43,7 @@
       </visual>
       <collision>
-        <origin xyz="0.035 0 0" rpy="1.57 1.57 0.0"/>
+       <origin xyz="0.0 0.0 0.0" rpy="0.0 0.0 0.0"/>
         <geometry>
-          <box size="0.03 0.15 0.03"/>
+          <box size="0.01905 0.1335 0.0222"/>
           <!-- <mesh filename="package://raw_description/meshes/cameras/sr300_optical_link.STL"/> -->
         </geometry>
@@ -48,5 +52,5 @@
     <!-- 1(1) rgb_frame -->
     <joint name="${name}_rgb_frame_joint" type="fixed">
-      <origin xyz="0.0 0.0 0.0" rpy="${frame_joint_rpy}" />
+      <origin xyz="${frame_joint_xyz}" rpy="${frame_joint_rpy}" />
       <parent link="${name}_link"/>
       <child link="${name}_rgb_frame"/>
@@ -66,5 +70,5 @@
     <!-- 2(1) depth_frame -->
     <joint name="${name}_depth_frame_joint" type="fixed">
-      <origin xyz="0.0 0.0 0.0" rpy="${frame_joint_rpy}" />
+      <origin xyz="${frame_joint_xyz}" rpy="${frame_joint_rpy}" />
       <parent link="${name}_link"/>
       <child link="${name}_depth_frame"/>
@@ -84,5 +88,5 @@
     <!-- 3(1) ir_frame -->
     <joint name="${name}_ir_frame_joint" type="fixed">
-      <origin xyz="0.0 0.0 0.0" rpy="${frame_joint_rpy}" />
+      <origin xyz="${frame_joint_xyz}" rpy="${frame_joint_rpy}" />
       <parent link="${name}_link"/>
       <child link="${name}_ir_frame"/>

Commit message: add sim camera to real run also

File: cob_description/urdf/sensors/r200.gazebo.xacro (robot description, xacro)
@@ -4,5 +4,5 @@
   <!-- use default values of realsense_camera/r200_nodelet_rgbd -->
   <xacro:macro name="r200_rgb_gazebo_v0" params="
-    name link_name frame_name camera_name visualize_wrist_camera_simulator
+    sim name link_name frame_name camera_name visualize_wrist_camera_simulator
     depth_fps:=30.0
     depth_height:=360
@@ -11,4 +11,10 @@
     color_height:=480
     color_width:=640" >
+    <xacro:if value="${sim}">
+      <xacro:property name="camera_name_sim" value="${camera_name}"/>
+    </xacro:if>
+    <xacro:unless value="${sim}">
+      <xacro:property name="camera_name_sim" value="${camera_name}_sim"/>
+    </xacro:unless>
     <gazebo reference="${link_name}">
       <!-- this camera sensor setup is copied from pr2 model in .gazebo/models/pr2/model.sdf -->
@@ -51,13 +57,13 @@
           <alwaysOn>true</alwaysOn>
           <updateRate>${color_fps}</updateRate>
-          <cameraName>${camera_name}_rgb_gazebo_simulation</cameraName>
+          <cameraName>${camera_name_sim}_rgb</cameraName>
           <frameName>${frame_name}</frameName>
-          <!-- <imageTopicName>/${camera_name}/rgb/image_raw</imageTopicName> -->
-          <imageTopicName>/${camera_name}/rgb/image_rect_color</imageTopicName>
-          <cameraInfoTopicName>/${camera_name}/rgb/camera_info</cameraInfoTopicName>
-          <!-- <depthImageTopicName>/${camera_name}/depth/image_raw</depthImageTopicName> -->
-          <depthImageTopicName>/${camera_name}/depth/image_rect</depthImageTopicName>
-          <depthImageCameraInfoTopicName>/${camera_name}/depth/camera_info</depthImageCameraInfoTopicName>
-          <pointCloudTopicName>/${camera_name}/depth_registered/points</pointCloudTopicName>
+          <!-- <imageTopicName>/${camera_name_sim}/rgb/image_raw</imageTopicName> -->
+          <imageTopicName>/${camera_name_sim}/rgb/image_rect_color</imageTopicName>
+          <cameraInfoTopicName>/${camera_name_sim}/rgb/camera_info</cameraInfoTopicName>
+          <!-- <depthImageTopicName>/${camera_name_sim}/depth/image_raw</depthImageTopicName> -->
+          <depthImageTopicName>/${camera_name_sim}/depth/image_rect</depthImageTopicName>
+          <depthImageCameraInfoTopicName>/${camera_name_sim}/depth/camera_info</depthImageCameraInfoTopicName>
+          <pointCloudTopicName>/${camera_name_sim}/depth_registered/points</pointCloudTopicName>
           <pointCloudCutoff>0.5</pointCloudCutoff>
           <pointCloudCutoffMax>5.0</pointCloudCutoffMax>
@@ -77,5 +83,5 @@
   <!-- https://github.com/PR2/pr2_common/blob/kinetic-devel/pr2_description/urdf/sensors/kinect2.gazebo.xacro -->
   <xacro:macro name="r200_ir_gazebo_v0" params="
-    name link_name frame_name camera_name visualize_wrist_camera_simulator
+    sim name link_name frame_name camera_name visualize_wrist_camera_simulator
     depth_fps:=30.0
     depth_height:=360
@@ -84,4 +90,10 @@
     color_height:=480
     color_width:=640" >
+    <xacro:if value="${sim}">
+      <xacro:property name="camera_name_sim" value="${camera_name}"/>
+    </xacro:if>
+    <xacro:unless value="${sim}">
+      <xacro:property name="camera_name_sim" value="${camera_name}_sim"/>
+    </xacro:unless>
     <gazebo reference="${link_name}">
       <sensor type="depth" name="${name}_ir_gazebo_simulation">
@@ -110,13 +122,13 @@
           <alwaysOn>true</alwaysOn>
           <updateRate>${color_fps}</updateRate>
-          <cameraName>${camera_name}_ir_gazebo_simulation</cameraName>
+          <cameraName>${camera_name_sim}_ir</cameraName>
           <frameName>${frame_name}</frameName>
-          <!-- <imageTopicName>/${camera_name}/ir/image_raw</imageTopicName> -->
-          <imageTopicName>/${camera_name}/ir/image_rect_ir</imageTopicName>
-          <cameraInfoTopicName>/${camera_name}/ir/camera_info</cameraInfoTopicName>
-          <!-- <depthImageTopicName>/${camera_name}/depth/image_raw</depthImageTopicName> -->
-          <depthImageTopicName>/${camera_name}/depth/image_rect</depthImageTopicName>
-          <depthImageCameraInfoTopicName>/${camera_name}/depth/camera_info</depthImageCameraInfoTopicName>
-          <pointCloudTopicName>/${camera_name}/depth/points</pointCloudTopicName>
+          <!-- <imageTopicName>/${camera_name_sim}/ir/image_raw</imageTopicName> -->
+          <imageTopicName>/${camera_name_sim}/ir/image_rect_ir</imageTopicName>
+          <cameraInfoTopicName>/${camera_name_sim}/ir/camera_info</cameraInfoTopicName>
+          <!-- <depthImageTopicName>/${camera_name_sim}/depth/image_raw</depthImageTopicName> -->
+          <depthImageTopicName>/${camera_name_sim}/depth/image_rect</depthImageTopicName>
+          <depthImageCameraInfoTopicName>/${camera_name_sim}/depth/camera_info</depthImageCameraInfoTopicName>
+          <pointCloudTopicName>/${camera_name_sim}/depth/points</pointCloudTopicName>
           <pointCloudCutoff>0.5</pointCloudCutoff>
           <pointCloudCutoffMax>5.0</pointCloudCutoffMax>

Commit message: remove sim camera to real run also

File: cob_description/urdf/sensors/r200.gazebo.xacro (robot description, xacro)
@@ -83,5 +83,5 @@
   <!-- https://github.com/PR2/pr2_common/blob/kinetic-devel/pr2_description/urdf/sensors/kinect2.gazebo.xacro -->
   <xacro:macro name="r200_ir_gazebo_v0" params="
-    sim name link_name frame_name camera_name visualize_wrist_camera_simulator
+    name link_name frame_name camera_name visualize_wrist_camera_simulator
     depth_fps:=30.0
     depth_height:=360
@@ -90,10 +90,5 @@
     color_height:=480
     color_width:=640" >
-    <xacro:if value="${sim}">
-      <xacro:property name="camera_name_sim" value="${camera_name}"/>
-    </xacro:if>
-    <xacro:unless value="${sim}">
-      <xacro:property name="camera_name_sim" value="${camera_name}_sim"/>
-    </xacro:unless>
+    <xacro:property name="camera_name_sim" value="${camera_name}"/>
     <gazebo reference="${link_name}">
       <sensor type="depth" name="${name}_ir_gazebo_simulation">

Commit message: fix bug for sim

File: cob_description/urdf/sensors/r200.gazebo.xacro (robot description, xacro)
@@ -4,5 +4,5 @@
   <!-- use default values of realsense_camera/r200_nodelet_rgbd -->
   <xacro:macro name="r200_rgb_gazebo_v0" params="
-    sim name link_name frame_name camera_name visualize_wrist_camera_simulator
+    name link_name frame_name camera_name visualize_wrist_camera_simulator
     depth_fps:=30.0
     depth_height:=360
@@ -11,10 +11,5 @@
     color_height:=480
     color_width:=640" >
-    <xacro:if value="${sim}">
-      <xacro:property name="camera_name_sim" value="${camera_name}"/>
-    </xacro:if>
-    <xacro:unless value="${sim}">
-      <xacro:property name="camera_name_sim" value="${camera_name}_sim"/>
-    </xacro:unless>
+  	<xacro:property name="camera_name_sim" value="${camera_name}"/>
     <gazebo reference="${link_name}">
       <!-- this camera sensor setup is copied from pr2 model in .gazebo/models/pr2/model.sdf -->
