Commit message: add sim into ur10 and robotiq, so when real robot runs, we dont load gazebo controller

File: cob_description/urdf/robotiq_gripper/robotiq_s_gripper.urdf.xacro (robot description, xacro)
@@ -13,10 +13,10 @@
     <xacro:robotiq_hand prefix="${name}_" reflect="${reflect}"/>
     <!-- ros_control plugin -->
-    <gazebo>
-      <!--<plugin name="RobotiqHandPlugin" filename="libRobotiqHandPlugin.so">-->
-      <plugin name="RobotiqHandPluginSingleHand" filename="libRobotiqHandPluginSingleHand.so">
-        <side>left</side>
-      </plugin>
-    </gazebo>
+    <xacro:if value="$(arg sim)">
+      <gazebo>
+        <plugin name="RobotiqHandPluginSingleHand" filename="libRobotiqHandPluginSingleHand.so">
+        </plugin>
+      </gazebo>
+    </xacro:if>
   </xacro:macro>
 </robot>

File: cob_description/urdf/ur_arm/ur10_arm.urdf.xacro (robot description, xacro)
@@ -3,5 +3,5 @@
   <xacro:include filename="$(find cob_description)/urdf/common.xacro" />
   <xacro:include filename="$(find ur_description)/urdf/ur10.urdf.xacro" />
-  <xacro:macro name="ur10" params="parent name *origin">
+  <xacro:macro name="ur10" params="parent name sim *origin">
     <!-- mount the arm to the robot -->
     <joint name="${name}_base_joint" type="fixed" >
@@ -13,10 +13,12 @@
     <xacro:ur10_robot prefix="${name}_" joint_limited="true"/>
     <!-- ros_control plugin -->
-    <gazebo>
-      <plugin name="ros_control" filename="libhwi_switch_gazebo_ros_control.so">
-        <robotNamespace>${name}</robotNamespace>
-        <filterJointsParam>joint_names</filterJointsParam>
-      </plugin>
-    </gazebo>
+    <xacro:if value="$(arg sim)">
+      <gazebo>
+        <plugin name="ros_control" filename="libhwi_switch_gazebo_ros_control.so">
+          <robotNamespace>${name}</robotNamespace>
+          <filterJointsParam>joint_names</filterJointsParam>
+        </plugin>
+      </gazebo>
+    </xacro:if>
   </xacro:macro>
 </robot>

Commit message: change camera pos

File: cob_description/urdf/robotiq_gripper/robotiq_s_gripper.urdf.xacro (robot description, xacro)
@@ -11,19 +11,21 @@
     </joint>
     <xacro:robotiq_hand prefix="${name}_" reflect="${reflect}" />
-    <gazebo>
-      <!-- The plugin is located at `./src/robotiq/robotiq_s_model_articulated_gazebo_plugins/include/robotiq_s_model_articulated_gazebo_plugins/RobotiqHandPluginSingleHand_controlMsg.h`. -->
-      <!-- We use this plugin instead of `RobotiqHandPluginSingleHand.h` so that we will publish msg type = `robotiq_s_model_control/SModel_robot_input` and `robotiq_s_model_control/SModel_robot_output` to topics `/SModelRobotInput` and `/SModelRobotOutput` to control BOTH the real and simulated gripper.  -->
-      <!-- If we use `RobotiqHandPluginSingleHand.h`, then we are publishing the msg type = `robotiq_s_model_articulated_msgs/SModelRobotInput` and `robotiq_s_model_articulated_msgs/SModelRobotOutput`. This is fine with simulation, but not real run. Not sure though. -->
-      <plugin name="RobotiqHandPluginSingleHand_controlMsg" filename="libRobotiqHandPluginSingleHand_controlMsg.so">
-        <!-- params from drc_sim in gazebo4 -->
-        <!-- http://gazebosim.org/tutorials?tut=drcsim_robotiq_hand&cat= -->
-        <!-- <kp_position>10.0</kp_position> -->
-        <!-- <kd_position>0.5</kd_position> -->
-        <!-- params from ros-industrial/robotiq in gazebo2 -->
-        <kp_position>1.0</kp_position>
-        <ki_position>0.0</ki_position>
-        <kd_position>0.5</kd_position>
-      </plugin>
-    </gazebo>
+    <xacro:if value="$(arg sim)">
+      <gazebo>
+        <!-- The plugin is located at `./src/robotiq/robotiq_s_model_articulated_gazebo_plugins/include/robotiq_s_model_articulated_gazebo_plugins/RobotiqHandPluginSingleHand_controlMsg.h`. -->
+        <!-- We use this plugin instead of `RobotiqHandPluginSingleHand.h` so that we will publish msg type = `robotiq_s_model_control/SModel_robot_input` and `robotiq_s_model_control/SModel_robot_output` to topics `/SModelRobotInput` and `/SModelRobotOutput` to control BOTH the real and simulated gripper.  -->
+        <!-- If we use `RobotiqHandPluginSingleHand.h`, then we are publishing the msg type = `robotiq_s_model_articulated_msgs/SModelRobotInput` and `robotiq_s_model_articulated_msgs/SModelRobotOutput`. This is fine with simulation, but not real run. Not sure though. -->
+        <plugin name="RobotiqHandPluginSingleHand_controlMsg" filename="libRobotiqHandPluginSingleHand_controlMsg.so">
+          <!-- params from drc_sim in gazebo4 -->
+          <!-- http://gazebosim.org/tutorials?tut=drcsim_robotiq_hand&cat= -->
+          <!-- <kp_position>10.0</kp_position> -->
+          <!-- <kd_position>0.5</kd_position> -->
+          <!-- params from ros-industrial/robotiq in gazebo2 -->
+          <kp_position>1.0</kp_position>
+          <ki_position>0.0</ki_position>
+          <kd_position>0.5</kd_position>
+        </plugin>
+      </gazebo>
+    </xacro:if>
   </xacro:macro>
 </robot>

File: cob_description/urdf/sensors/realsense.urdf.xacro (robot description, xacro)
@@ -41,5 +41,5 @@
       </visual>
       <collision>
-        <origin xyz="-0.025 0.0 -0.01" rpy="0.0 0.0 0.0"/>
+        <origin xyz="0 -0.01 -0.03" rpy="1.57 1.57 0.0"/>
         <geometry>
           <!-- <box size="0.007 0.130 0.0118"/> -->

Commit message: using irg-jade of robotiq

File: cob_description/urdf/robotiq_gripper/robotiq_s_gripper.urdf.xacro (robot description, xacro)
@@ -4,11 +4,20 @@
   <xacro:include filename="$(find robotiq_s_model_visualization)/cfg/robotiq_hand_macro.urdf.xacro" />
   <xacro:macro name="robotiq" params="parent name reflect sim *origin">
+  	<!-- If we use irg-raw3-6 branch of https://github.com/Shentheman/robotiq -->
     <!-- mount the gripper to the arm -->
-    <joint name="${name}_robotiq_hand_joint" type="fixed">
+    <!-- <joint name="${name}_robotiq_hand_joint" type="fixed">
       <xacro:insert_block name="origin"/>
       <parent link="${parent}"/>
       <child link="${name}_palm"/>
     </joint>
-    <xacro:robotiq_hand prefix="${name}_" reflect="${reflect}" />
+    <xacro:robotiq_hand prefix="${name}_" reflect="${reflect}" /> -->
+  	<!-- If we use irg-jade branch of https://github.com/Shentheman/robotiq -->
+    <xacro:include filename="$(find robotiq_s_model_visualization)/cfg/robotiq_hand_macro.urdf.xacro" />
+    <xacro:robotiq_hand
+      prefix="${name}_"
+      parent="${parent}"
+      reflect="-1">
+      <xacro:insert_block name="origin"/>
+    </xacro:robotiq_hand>
     <xacro:if value="$(arg sim)">
       <gazebo>

Commit message: add FT sensor

File: cob_description/urdf/robotiq_gripper/robotiq_s_gripper.urdf.xacro (robot description, xacro)
@@ -4,5 +4,5 @@
   <xacro:include filename="$(find robotiq_s_model_visualization)/cfg/robotiq_hand_macro.urdf.xacro" />
   <xacro:macro name="robotiq" params="parent name reflect sim *origin">
-  	<!-- If we use irg-raw3-6 branch of https://github.com/Shentheman/robotiq -->
+    <!-- If we use irg-raw3-6 branch of https://github.com/Shentheman/robotiq -->
     <!-- mount the gripper to the arm -->
     <!-- <joint name="${name}_robotiq_hand_joint" type="fixed">
@@ -12,9 +12,39 @@
     </joint>
     <xacro:robotiq_hand prefix="${name}_" reflect="${reflect}" /> -->
-  	<!-- If we use irg-jade branch of https://github.com/Shentheman/robotiq -->
+    <!-- If we use irg-jade branch of https://github.com/Shentheman/robotiq -->
     <xacro:include filename="$(find robotiq_s_model_visualization)/cfg/robotiq_hand_macro.urdf.xacro" />
+    <!-- ===================================== -->
+    <!-- FT sensor rough size = box = 0.05 x 0.05 x 0.03 -->
+    <!-- add a link bw arm_wrist_3_link and gripper_palm -->
+    <joint name="$arm_tool0_2_FT_sensor" type="fixed">
+      <!-- length of the FT sensor = 0.03 -->
+      <origin xyz="0 0 0.03" rpy="0 0 0" />
+      <parent link="${parent}"/>
+      <child link="${name}_FT_sensor"/>
+    </joint>
+    <link name="${name}_FT_sensor" >
+      <inertial>
+        <mass value="0.1" />
+        <origin xyz="0.0 0.0 0.0" rpy="0.0 0.0 0.0" />
+        <inertia ixx="0.0" ixy="0.0" ixz="0.0" iyy="0.0" iyz="0.0" izz="0.0" />
+      </inertial>
+      <visual>
+        <!-- length of the FT sensor / 2 = 0.03 / 2-->
+       <origin xyz="0.0 0.0 -0.015" rpy="0.0 0.0 0.0"/>
+        <geometry>
+          <box size="0.05 0.05 0.03"/>
+        </geometry>
+      </visual>
+      <collision>
+       <origin xyz="0.0 0.0 -0.015" rpy="0.0 0.0 0.0"/>
+        <geometry>
+          <box size="0.05 0.05 0.03"/>
+        </geometry>
+      </collision>
+    </link>
+    <!-- ===================================== -->
     <xacro:robotiq_hand
       prefix="${name}_"
-      parent="${parent}"
+      parent="${name}_FT_sensor"
       reflect="-1">
       <xacro:insert_block name="origin"/>
